Commit message: Initiating the Dynamic Modelling into Urdf

File: autodrive_devkit/ws/src/f1tenth_description/urdf/f1tenth_car.urdf.xacro (robot description, xacro)
@@ -2,19 +2,19 @@
 <robot name="f1tenth_car" xmlns:xacro="http://ros.org/wiki/xacro">
   <!-- Propriedades (dimensões) em metros -->
-  <xacro:property name="wheel_radius" value="0.034"/>       <!-- 3.4 cm :contentReference[oaicite:5]{index=5} -->
-  <xacro:property name="wheel_width"  value="0.023"/>       <!-- 2.3 cm :contentReference[oaicite:6]{index=6} -->
-  <xacro:property name="half_wheelbase" value="0.13"/>      <!-- Metade de 26 cm :contentReference[oaicite:7]{index=7} -->
-  <xacro:property name="half_track" value="0.0835"/>        <!-- Metade de ~16.7 cm (centro a centro das rodas) -->
-  <xacro:property name="chassis_length" value="0.38"/>      <!-- 38 cm :contentReference[oaicite:8]{index=8} -->
-  <xacro:property name="chassis_width"  value="0.125"/>     <!-- 12.5 cm :contentReference[oaicite:9]{index=9} -->
-  <xacro:property name="chassis_thickness" value="0.014"/>  <!-- 1.4 cm :contentReference[oaicite:10]{index=10} -->
-  <xacro:property name="top_chassis_width" value="0.101"/>  <!-- 10.1 cm :contentReference[oaicite:11]{index=11} -->
-  <xacro:property name="top_chassis_thickness" value="0.002"/> <!-- 0.2 cm :contentReference[oaicite:12]{index=12} -->
-  <xacro:property name="ground_clearance" value="0.003"/>   <!-- 0.3 cm do chão ao chassi inferior :contentReference[oaicite:13]{index=13} -->
-  <xacro:property name="top_chassis_height" value="0.069"/> <!-- 6.9 cm do chão ao topo do chassi sup. :contentReference[oaicite:14]{index=14} -->
-  <xacro:property name="lidar_diameter" value="0.038"/>     <!-- 3.8 cm :contentReference[oaicite:15]{index=15} -->
-  <xacro:property name="lidar_height" value="0.07"/>        <!-- 7 cm :contentReference[oaicite:16]{index=16} -->
-  <xacro:property name="lidar_offset_x" value="0.10"/>      <!-- ~9 cm atrás do para-choque frontal (0.19-0.10 = 0.09 m):contentReference[oaicite:17]{index=17} -->
-  <xacro:property name="lidar_base_z" value="0.073"/>       <!-- Base do LiDAR ~0.4 cm acima do topo do chassi sup. (para altura total ~14.3 cm):contentReference[oaicite:18]{index=18} -->
+  <xacro:property name="wheel_radius" value="0.034"/>       <!-- 3.4 cm -->
+  <xacro:property name="wheel_width"  value="0.023"/>       <!-- 2.3 cm -->
+  <xacro:property name="half_wheelbase" value="0.13"/>      <!-- L total = 0.26 m -->
+  <xacro:property name="half_track" value="0.0835"/>        <!-- ~16.7 cm / 2 -->
+  <xacro:property name="chassis_length" value="0.38"/>      <!-- 38 cm -->
+  <xacro:property name="chassis_width"  value="0.125"/>     <!-- 12.5 cm -->
+  <xacro:property name="chassis_thickness" value="0.014"/>  <!-- 1.4 cm -->
+  <xacro:property name="top_chassis_width" value="0.101"/>  <!-- 10.1 cm -->
+  <xacro:property name="top_chassis_thickness" value="0.002"/> <!-- 0.2 cm -->
+  <xacro:property name="ground_clearance" value="0.003"/>   <!-- 0.3 cm -->
+  <xacro:property name="top_chassis_height" value="0.069"/> <!-- 6.9 cm -->
+  <xacro:property name="lidar_diameter" value="0.038"/>     <!-- 3.8 cm -->
+  <xacro:property name="lidar_height" value="0.07"/>        <!-- 7 cm -->
+  <xacro:property name="lidar_offset_x" value="0.10"/>      <!-- ~0.09 m atrás da dianteira -->
+  <xacro:property name="lidar_base_z" value="0.073"/>       <!-- base do LiDAR -->
   <!-- Link principal do chassi (base_link) -->
   <link name="base_link">
@@ -36,16 +36,15 @@
       </geometry>
       <material name="TransparentBlue">
-        <color rgba="0.3 0.5 1.0 0.5"/>  <!-- azul translúcido -->
-      </material>
-    </visual>
-    <!-- Geometria de colisão (opcional, usando caixa englobante do chassi inteiro) -->
+        <color rgba="0.3 0.5 1.0 0.5"/>
+      </material>
+    </visual>
+    <!-- Geometria de colisão (caixa englobante) -->
     <collision>
       <origin xyz="0 0 ${ground_clearance + (top_chassis_height)/2}" rpy="0 0 0"/>
       <geometry>
-        <!-- Caixa cobrindo todo o volume do robô aproximado -->
         <box size="${chassis_length} ${chassis_width} ${top_chassis_height}"/>
       </geometry>
     </collision>
-    <!-- Inércia aproximada do chassi (massa ~2 kg distribuída) -->
+    <!-- Inércia aproximada do chassi (massa ~2 kg) -->
     <inertial>
       <mass value="2.0"/>
@@ -54,9 +53,37 @@
     </inertial>
   </link>
-  <!-- Links e juntas para as 4 rodas -->
-  <!-- Roda Dianteira Esquerda -->
+  <!-- ========== MANGAS DE EIXO (esterço dianteiro) ========== -->
+  <link name="steer_front_left_link">
+    <inertial>
+      <mass value="0.02"/>
+      <origin xyz="0 0 0"/>
+      <inertia ixx="1e-4" ixy="0" ixz="0" iyy="1e-4" iyz="0" izz="1e-4"/>
+    </inertial>
+  </link>
+  <joint name="joint_steer_front_left" type="revolute">
+    <parent link="base_link"/>
+    <child link="steer_front_left_link"/>
+    <origin xyz="${half_wheelbase} ${half_track} ${wheel_radius}" rpy="0 0 0"/>
+    <axis xyz="0 0 1"/>
+    <limit effort="5.0" lower="-0.7" upper="0.7" velocity="2.0"/>
+  </joint>
+  <link name="steer_front_right_link">
+    <inertial>
+      <mass value="0.02"/>
+      <origin xyz="0 0 0"/>
+      <inertia ixx="1e-4" ixy="0" ixz="0" iyy="1e-4" iyz="0" izz="1e-4"/>
+    </inertial>
+  </link>
+  <joint name="joint_steer_front_right" type="revolute">
+    <parent link="base_link"/>
+    <child link="steer_front_right_link"/>
+    <origin xyz="${half_wheelbase} -${half_track} ${wheel_radius}" rpy="0 0 0"/>
+    <axis xyz="0 0 1"/>
+    <limit effort="5.0" lower="-0.7" upper="0.7" velocity="2.0"/>
+  </joint>
+  <!-- ========== Rodas ========== -->
+  <!-- Dianteira Esquerda -->
   <link name="wheel_front_left">
     <visual>
-      <!-- Cylinder axis along Y (rotate 90deg about X to align eixo de rotação) -->
       <origin xyz="0 0 0" rpy="1.5708 0 0"/>
       <geometry>
@@ -80,10 +107,10 @@
   </link>
   <joint name="joint_wheel_front_left" type="continuous">
-    <parent link="base_link"/>
+    <parent link="steer_front_left_link"/>
     <child link="wheel_front_left"/>
-    <origin xyz="${half_wheelbase} ${half_track} ${wheel_radius}" rpy="0 0 0"/>
-    <axis xyz="0 1 0"/>  <!-- eixo de rotação: eixo Y (esquerda-direita) -->
-  </joint>
-  <!-- Roda Dianteira Direita -->
+    <origin xyz="0 0 0" rpy="0 0 0"/>
+    <axis xyz="0 1 0"/>
+  </joint>
+  <!-- Dianteira Direita -->
   <link name="wheel_front_right">
     <visual>
@@ -107,10 +134,10 @@
   </link>
   <joint name="joint_wheel_front_right" type="continuous">
-    <parent link="base_link"/>
+    <parent link="steer_front_right_link"/>
     <child link="wheel_front_right"/>
-    <origin xyz="${half_wheelbase} -${half_track} ${wheel_radius}" rpy="0 0 0"/>
-    <axis xyz="0 1 0"/>
-  </joint>
-  <!-- Roda Traseira Esquerda -->
+    <origin xyz="0 0 0" rpy="0 0 0"/>
+    <axis xyz="0 1 0"/>
+  </joint>
+  <!-- Traseira Esquerda -->
   <link name="wheel_rear_left">
     <visual>
@@ -139,5 +166,5 @@
     <axis xyz="0 1 0"/>
   </joint>
-  <!-- Roda Traseira Direita -->
+  <!-- Traseira Direita -->
   <link name="wheel_rear_right">
     <visual>
@@ -166,5 +193,5 @@
     <axis xyz="0 1 0"/>
   </joint>
-  <!-- Link do LiDAR (sensor no topo frontal) -->
+  <!-- Link do LiDAR -->
   <link name="laser_link">
     <visual>
@@ -194,7 +221,6 @@
     <origin xyz="${lidar_offset_x} 0 ${lidar_base_z}" rpy="0 0 0"/>
   </joint>
-  <!-- Link da IMU (fixo no chassi, centro do robô) -->
+  <!-- Link da IMU -->
   <link name="imu_link">
-    <!-- sem geometria visual -->
     <inertial>
       <mass value="0.01"/>
@@ -208,3 +234,18 @@
     <origin xyz="0 0 ${top_chassis_height/2}" rpy="0 0 0"/>
   </joint>
+  <!-- ============= GAZEBO: Plugin Dynamic-Actuator ============= -->
+  <gazebo>
+    <plugin name="f1tenth_interface_plugin" filename="libf1tenth_interface_plugin.so">
+      <steer_fl_joint>joint_steer_front_left</steer_fl_joint>
+      <steer_fr_joint>joint_steer_front_right</steer_fr_joint>
+      <wheel_rl_joint>joint_wheel_rear_left</wheel_rl_joint>
+      <wheel_rr_joint>joint_wheel_rear_right</wheel_rr_joint>
+      <steer_topic>/autodrive/f1tenth_1/steering_command</steer_topic>
+      <throttle_topic>/autodrive/f1tenth_1/throttle_command</throttle_topic>
+      <brake_topic>/autodrive/f1tenth_1/brake_command</brake_topic>
+      <k_speed>2.0</k_speed>                 <!-- m/s @ 100% throttle -->
+      <wheel_radius>0.034</wheel_radius>
+      <steer_limit_rad>0.698</steer_limit_rad> <!-- ~40° -->
+    </plugin>
+  </gazebo>
 </robot>

Commit message: Fixed imu orientation, added camera, added conf files for mapping, plan and control

File: autodrive_devkit/ws/src/f1tenth_description/urdf/f1tenth_car.urdf.xacro (robot description, xacro)
@@ -234,4 +234,27 @@
     <child link="imu_link"/>
     <origin xyz="0 0 ${top_chassis_height/2}" rpy="0 0 0"/>
+  </joint>
+  <!-- ========== RGB-D CAMERA (para RTAB-MAP) ========== -->
+  <link name="front_camera_link">
+    <visual>
+      <origin xyz="0 0 0" rpy="0 0 0"/>
+      <geometry>
+        <box size="0.03 0.03 0.03"/>
+      </geometry>
+      <material name="DarkGray">
+        <color rgba="0.2 0.2 0.2 1.0"/>
+      </material>
+    </visual>
+    <inertial>
+      <mass value="0.02"/>
+      <origin xyz="0 0 0" rpy="0 0 0"/>
+      <inertia ixx="1e-5" ixy="0" ixz="0" iyy="1e-5" iyz="0" izz="1e-5"/>
+    </inertial>
+  </link>
+  <joint name="joint_front_camera" type="fixed">
+    <parent link="base_link"/>
+    <child link="front_camera_link"/>
+    <!-- Movida mais à frente do LIDAR -->
+    <origin xyz="${lidar_offset_x + 0.075} 0 ${lidar_base_z - 0.02}" rpy="0 0 0"/>
   </joint>
     <!-- ======== GAZEBO: SENSOR LiDAR NO laser_link (publica /scan) ======== -->
@@ -332,4 +355,55 @@
     </sensor>
   </gazebo>
+  <!-- Sensor de câmera RGB-D -->
+  <gazebo reference="front_camera_link">
+    <!-- Câmera RGB -->
+    <sensor name="front_camera_rgb" type="camera">
+      <always_on>true</always_on>
+      <update_rate>30.0</update_rate>
+      <camera>
+        <horizontal_fov>1.3962634</horizontal_fov> <!-- ~80° -->
+        <image>
+          <width>640</width>
+          <height>480</height>
+          <format>R8G8B8</format>
+        </image>
+        <clip>
+          <near>0.02</near>
+          <far>50.0</far>
+        </clip>
+      </camera>
+      <plugin name="front_camera_rgb_plugin" filename="libgazebo_ros_camera.so">
+        <ros>
+          <remapping>~/image_raw:=/autodrive/f1tenth_1/front_camera/image_raw</remapping>
+          <remapping>~/camera_info:=/autodrive/f1tenth_1/front_camera/camera_info</remapping>
+        </ros>
+        <frame_name>front_camera_link</frame_name>
+      </plugin>
+    </sensor>
+    <!-- Câmera Depth (simulada via sensor de profundidade) -->
+    <sensor name="front_camera_depth" type="depth">
+      <always_on>true</always_on>
+      <update_rate>30.0</update_rate>
+      <camera>
+        <horizontal_fov>1.3962634</horizontal_fov>
+        <image>
+          <width>640</width>
+          <height>480</height>
+          <format>FLOAT32</format>
+        </image>
+        <clip>
+          <near>0.05</near>
+          <far>20.0</far>
+        </clip>
+      </camera>
+      <plugin name="front_camera_depth_plugin" filename="libgazebo_ros_depth_camera.so">
+        <ros>
+          <remapping>~/image_raw:=/autodrive/f1tenth_1/front_camera/depth/image_raw</remapping>
+          <remapping>~/camera_info:=/autodrive/f1tenth_1/front_camera/depth/camera_info</remapping>
+        </ros>
+        <frame_name>front_camera_link</frame_name>
+      </plugin>
+    </sensor>
+  </gazebo>
   <gazebo>
     <plugin name="f1tenth_ackermann" filename="libgazebo_ros_ackermann_drive.so">
@@ -354,18 +428,3 @@
     </plugin>
   </gazebo>
-  <!-- ============= GAZEBO: Plugin Dynamic-Actuator ============= -->
-  <gazebo>
-    <plugin name="f1tenth_interface_plugin" filename="libf1tenth_interface_plugin.so">
-      <steer_fl_joint>joint_steer_front_left</steer_fl_joint>
-      <steer_fr_joint>joint_steer_front_right</steer_fr_joint>
-      <wheel_rl_joint>joint_wheel_rear_left</wheel_rl_joint>
-      <wheel_rr_joint>joint_wheel_rear_right</wheel_rr_joint>
-      <steer_topic>/autodrive/f1tenth_1/steering_command</steer_topic>
-      <throttle_topic>/autodrive/f1tenth_1/throttle_command</throttle_topic>
-      <brake_topic>/autodrive/f1tenth_1/brake_command</brake_topic>
-      <k_speed>2.0</k_speed>                 <!-- m/s @ 100% throttle -->
-      <wheel_radius>0.034</wheel_radius>
-      <steer_limit_rad>0.698</steer_limit_rad> <!-- ~40° -->
-    </plugin>
-  </gazebo>
 </robot>

Commit message: Enabled Global and Local Costmap using main launch and slam toolbox launch

File: autodrive_devkit/ws/src/f1tenth_description/urdf/f1tenth_car.urdf.xacro (robot description, xacro)
@@ -17,4 +17,11 @@
   <xacro:property name="lidar_offset_x" value="0.10"/>      <!-- ~0.09 m atrás da dianteira -->
   <xacro:property name="lidar_base_z" value="0.073"/>       <!-- base do LiDAR -->
+  <!-- ===== Novo frame raiz 2D ===== -->
+  <link name="base_footprint"/>
+  <joint name="base_footprint_to_base_link" type="fixed">
+    <parent link="base_footprint"/>
+    <child  link="base_link"/>
+    <origin xyz="0 0 0" rpy="0 0 0"/>
+  </joint>
   <!-- Link principal do chassi (base_link) -->
   <link name="base_link">
@@ -258,5 +265,5 @@
     <origin xyz="${lidar_offset_x + 0.075} 0 ${lidar_base_z - 0.02}" rpy="0 0 0"/>
   </joint>
-    <!-- ======== GAZEBO: SENSOR LiDAR NO laser_link (publica /scan) ======== -->
+  <!-- ======== GAZEBO: SENSOR LiDAR NO laser_link (publica /scan) ======== -->
   <gazebo reference="laser_link">
     <sensor name="lidar_sensor" type="ray">
@@ -423,7 +430,7 @@
       <!-- ativa publicação de odom e TF -->
       <publish_odom>true</publish_odom>
-      <publish_odom_tf>false</publish_odom_tf>
+      <publish_odom_tf>true</publish_odom_tf>
       <odometry_frame>odom</odometry_frame>
-      <robot_base_frame>base_link</robot_base_frame>
+      <robot_base_frame>base_footprint</robot_base_frame>
     </plugin>
   </gazebo>
