Commit message: Path Planning Working, Control Working, Avoiding Obstacle

File: autodrive_devkit/ws/src/f1tenth_description/urdf/f1tenth_car.urdf (robot description, URDF)
Before this commit: robot f1tenth_car, 11 links, 10 joints
Links:
- link base_link: geometry collision box size=0.38 0.125 0.069; visual box size=0.38 0.101 0.002
- link laser_link: geometry collision cylinder length=0.07 radius=0.019; visual cylinder length=0.07 radius=0.019
- link wheel_front_left: geometry collision cylinder length=0.023 radius=0.034; visual cylinder length=0.023 radius=0.034
- link wheel_front_right: geometry collision cylinder length=0.023 radius=0.034; visual cylinder length=0.023 radius=0.034
- link wheel_rear_left: geometry collision cylinder length=0.023 radius=0.034; visual cylinder length=0.023 radius=0.034
- link wheel_rear_right: geometry collision cylinder length=0.023 radius=0.034; visual cylinder length=0.023 radius=0.034
Joints:
- joint joint_front_camera: origin xyz=${lidar_offset_x + 0.075} 0 ${lidar_base_z - 0.02} rpy=0 0 0 -> xyz=0.175 0 0.05299999999999999 rpy=0 0 0
- joint joint_imu: origin xyz=0 0 ${top_chassis_height/2} rpy=0 0 0 -> xyz=0 0 0.0345 rpy=0 0 0
- joint joint_laser: origin xyz=${lidar_offset_x} 0 ${lidar_base_z} rpy=0 0 0 -> xyz=0.1 0 0.073 rpy=0 0 0
- joint joint_steer_front_left: origin xyz=${half_wheelbase} ${half_track} ${wheel_radius} rpy=0 0 0 -> xyz=0.13 0.0835 0.034 rpy=0 0 0
- joint joint_steer_front_right: origin xyz=${half_wheelbase} -${half_track} ${wheel_radius} rpy=0 0 0 -> xyz=0.13 -0.0835 0.034 rpy=0 0 0
- joint joint_wheel_rear_left: origin xyz=-${half_wheelbase} ${half_track} ${wheel_radius} rpy=0 0 0 -> xyz=-0.13 0.0835 0.034 rpy=0 0 0
- joint joint_wheel_rear_right: origin xyz=-${half_wheelbase} -${half_track} ${wheel_radius} rpy=0 0 0 -> xyz=-0.13 -0.0835 0.034 rpy=0 0 0
